File: ESP32_board.kicad_pcb (KiCad board)
At the start: 4 copper layers, 92 x 54.6 mm, 89 parts, among them J1 SS-52400-002, J2 B2B-PH-SM4-TB, J3 GSD090012SEU, J4 Conn_01x04_Pin, J5 Conn_01x05_Pin, Q1 TEMT6000X01, Q2 BC817, Q3 BC817, U1 MCP73871, U2 BME280, U3 ESP32-C3-WROOM-02-H4, U4 CP2102N-Axx-xQFN20, U5 USBLC6-2SC6, U6 W25Q32JVSSIQ, U7 MAX4466EXK

Commit message: finished routing
Parts:
- moved R5 4.37 mm to (177.0, 120.7)
- moved R6 4.37 mm to (179.3, 120.7)
- moved R1 4.33 mm to (177.0, 124.7)
- moved R2 4.08 mm to (179.3, 124.7)
- moved Q1 2.03 mm to (204.7, 107.9)
- moved R23 1.27 mm to (205.7, 105.3)
- moved F1 0.68 mm to (188.7, 120.2)
- moved U1 0.63 mm to (181.0, 129.9)
- moved R32 0.51 mm to (205.7, 129.5)
- moved U5 0.51 mm to (195.1, 119.9)
- turned C21 to 180 degrees
- turned R12 to 0 degrees
Routing:
- net GND: track 25.4 -> 135.0 mm, vias 22 -> 49
- net /ESP32-C3-02/RX_TX: track 0.00 -> 83.3 mm, vias 0 -> 2
- net /ESP32-C3-02/TX_RX: track 0.00 -> 83.2 mm, vias 0 -> 2
- net /ESP32-C3-02/GPIO19: track 0.00 -> 81.5 mm, vias 0 -> 4
- net /ESP32-C3-02/EN: track 0.00 -> 79.1 mm, vias 0 -> 2
- net /ESP32-C3-02/GPIO18: track 0.00 -> 77.8 mm, vias 0 -> 2
- net /ESP32-C3-02/PHOTO_C: track 0.00 -> 62.0 mm, vias 0 -> 2
- net /ESP32-C3-02/GPIO8: track 0.00 -> 61.6 mm, vias 0 -> 2
- net +3V3: track 16.5 -> 77.1 mm, vias 12 -> 30
- net /ESP32-C3-02/BOOT: track 0.00 -> 56.8 mm, vias 0 -> 2
- net /ESP32-C3-02/MIC_OUT: track 0.00 -> 45.2 mm
- net /ESP32-C3-02/RTS: track 0.00 -> 36.3 mm, vias 0 -> 2
- net /ESP32-C3-02/DTR: track 0.00 -> 36.3 mm, vias 0 -> 3
- net /CHARGING: track 0.00 -> 24.2 mm, vias 0 -> 2
- net Net-(U4-VBUS): track 0.00 -> 20.7 mm
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
Commit message: corrected boot control schematic and layout
Parts:
- added C23: 0.1u, Capacitor_SMD:C_0805_2012Metric, F.Cu at (208.7, 109.0)
- added C24: 10n, Capacitor_SMD:C_0805_2012Metric, F.Cu at (201.7, 104.4)
- added C25: 10n, Capacitor_SMD:C_0805_2012Metric, F.Cu at (199.3, 104.4)
Connections:
- Q1 pad 1: GND -> /ESP32-C3-02/PHOTO_C
- Q1 pad 3: /ESP32-C3-02/PHOTO_C -> +3V3
- Q3 pad 2: /ESP32-C3-02/BOOT -> /ESP32-C3-02/DTR
- Q3 pad 3: /ESP32-C3-02/DTR -> /ESP32-C3-02/BOOT
- R23 pad 1: +3V3 -> /ESP32-C3-02/PHOTO_C
- R23 pad 2: /ESP32-C3-02/PHOTO_C -> GND
- U3 pad 18: /ESP32-C3-02/CS_SD -> /ESP32-C3-02/MIC_OUT
- U3 pad 4: /ESP32-C3-02/MIC_OUT -> /ESP32-C3-02/CS_SD
Routing:
- net /ESP32-C3-02/MIC_OUT: track 45.2 -> 64.3 mm, vias 0 -> 2
- net /ESP32-C3-02/PHOTO_C: track 62.0 -> 72.2 mm
- net GND: track 135.0 -> 138.7 mm, vias 49 -> 51
- net /ESP32-C3-02/DTR: track 36.3 -> 40.0 mm
- net /ESP32-C3-02/BOOT: track 56.8 -> 60.3 mm
- net +3V3: track 77.1 -> 80.3 mm
- net /ESP32-C3-02/CS_SD: track 27.9 -> 29.8 mm

Commit message: added pot to mic amp, made buttons bigger
Parts:
- removed REF** (x3): MountingHole_2.5mm, MountingHole:MountingHole_2.5mm
- added R17: 35WR100KLFTR, ESP32_project_Footprints:TRIM_35WR100KLFTR, F.Cu at (204.1, 97.0)
